File: design-files/schematics/output-shift-register-wiring/output-shift-register-wiring.kicad_sch (KiCad schematic)
At the start: 48 parts, among them U1 74HC595, U2 TLC5917, U3 DM13A

Commit message: Update 74HC595 schematic (#245)
* Update schematic

* Update 74HC595 schematic and pin mappings

* Fix pin number
Connections:
- net CLOCK: now also U1.11 (SRCLK); no longer U1.12 (RCLK)
- net LATCH: now also U1.12 (RCLK); no longer U1.11 (SRCLK)
Changed lines of the file:
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@@
 (kicad_sch
-	(version 20231120)
+	(version 20250114)
 	(generator "eeschema")
-	(generator_version "8.0")
+	(generator_version "9.0")
 	(paper "A4")
+	(text "220\nresistors"
+		(exclude_from_sim no)
+		(at 90.424 26.162 0)
+		(effects
+			(font
+				(size 1.27 1.27)
+			)
+		)
+	)
+	(text "Dedicated +5V power,\nnot from a +5V pin on the board."
+		(exclude_from_sim no)
+		(at 208.026 16.51 0)
+		(effects
+			(font
+				(size 1.27 1.27)
+			)
+		)
+	)
+	(text "Dedicated +5V power,\nnot from a +5V pin on the board."
+		(exclude_from_sim no)
+		(at 58.42 16.51 0)
+		(effects
+			(font
+				(size 1.27 1.27)
+			)
+		)
+	)
+	(text "Dedicated +5V power,\nnot from a +5V pin on the board."
+		(exclude_from_sim no)
+		(at 140.716 16.51 0)
+		(effects
+			(font
+				(size 1.27 1.27)
+			)
+		)
+	)
 	(junction
 		(at 167.64 49.53)
@@
 		)
 	)
-	(text "220\nresistors"
-		(exclude_from_sim no)
-		(at 90.424 26.162 0)
-		(effects
-			(font
-				(size 1.27 1.27)
-			)
-		)
-	)
-	(text "Dedicated +5V power,\nnot from a +5V pin on the board."
-		(exclude_from_sim no)
-		(at 208.026 16.51 0)
-		(effects
-			(font
-				(size 1.27 1.27)
-			)
-		)
-	)
-	(text "Dedicated +5V power,\nnot from a +5V pin on the board."
-		(exclude_from_sim no)
-		(at 58.42 16.51 0)
-		(effects
-			(font
-				(size 1.27 1.27)
-			)
-		)
-	)
-	(text "Dedicated +5V power,\nnot from a +5V pin on the board."
-		(exclude_from_sim no)
-		(at 140.716 16.51 0)
-		(effects
-			(font
-				(size 1.27 1.27)
-			)
-		)
-	)
 	(label "CLOCK"
 		(at 189.23 36.83 0)
@@
 		)
 	)
-	(label "LATCH"
+	(label "CLOCK"
 		(at 40.64 39.37 0)
 		(effects
@@
 		)
 	)
-	(label "CLOCK"
+	(label "LATCH"
 		(at 40.64 46.99 0)
 		(effects
@@
 		)
 	)
+	(embedded_fonts no)
 )
