File: design-files/schematics/seven-segment-displays/seven-segment-displays.kicad_sch (KiCad schematic)
At the start: 3 parts, among them U3 4-digit TM1637

Commit message: Fix +5V on MAX7219 diagram (#249)
Connections:
- net +5C is gone; now on net +5V: U1.1 (VCC), U2.1 (VCC)
